Commit message: fix keyboard teleop for wrist

File: stretch_description/urdf/stretch_dex_wrist_beta.xacro (robot description, xacro)
@@ -107,5 +107,5 @@
     <axis
       xyz="0 0 1" />
-    <limit effort="100" lower="-1.14" upper="3.14" velocity="1.0"/>
+    <limit effort="100" lower="-0.56" upper="1.56" velocity="1.0"/>
   </joint>
   <link

Commit message: ready for j2 test of dex_wrist

File: stretch_description/urdf/stretch_dex_wrist_beta.xacro (robot description, xacro)
@@ -106,6 +106,6 @@
       link="link_wrist_pitch" />
     <axis
-      xyz="0 0 1" />
-    <limit effort="100" lower="-0.56" upper="1.56" velocity="1.0"/>
+      xyz="0 0 -1" />
+    <limit effort="100" lower="-1.57" upper="0.56" velocity="1.0"/>
   </joint>
   <link
