Commit message: Mitski URDF xacros corrected

File: stretch_description/urdf/stretch_description.xacro (robot description, xacro)
@@ -4,5 +4,5 @@
   <!--<xacro:include filename="stretch_gripper_with_puller.xacro" />-->
   <!--<xacro:include filename="stretch_dry_erase_marker.xacro" />-->
-  <!--<xacro:include filename="stretch_main.xacro" />-->
+<!--  <xacro:include filename="stretch_main.xacro" />-->
   <xacro:include filename="stretch_mitski.xacro" />
   <xacro:include filename="stretch_aruco.xacro" />

File: stretch_description/urdf/stretch_mitski.xacro (robot description, xacro)
@@ -88,5 +88,5 @@
   <joint
     name="joint_right_wheel"
-    type="revolute">
+    type="continuous">
     <origin
       xyz="0 -0.17035 0.0508"
@@ -142,5 +142,5 @@
   <joint
     name="joint_left_wheel"
-    type="revolute">
+    type="continuous">
     <origin
       xyz="0 0.17035 0.0508"
@@ -153,4 +153,53 @@
       xyz="0 0 -1" />
     <dynamics damping="${joint_damping}" friction="${joint_friction}" spring_reference="${joint_spring_reference}" spring_stiffness="{joint_spring_stiffness}"/>
+  </joint>
+  <link name="caster_link">
+    <collision>
+      <geometry>
+        <sphere radius="0.032"/>
+      </geometry>
+      <origin rpy="0 0 0" xyz="0 0 0"/>
+      <surface>
+        <friction>
+          <ode>
+            <mu>0</mu>
+            <mu2>0</mu2>
+            <slip1>1.0</slip1>
+            <slip2>1.0</slip2>
+          </ode>
+        </friction>
+      </surface>
+    </collision>
+    <visual>
+      <origin
+        xyz="0 0 0"
+        rpy="0 0 0" />
+      <geometry>
+        <mesh
+          filename="package://stretch_description/meshes/omni_wheel_m.STL" />
+      </geometry>
+      <material
+        name="">
+        <color
+          rgba="0.792156862745098 0.819607843137255 0.933333333333333 1" />
+      </material>
+    </visual>
+    <inertial>
+      <mass value="0.01" />
+      <origin xyz="0 0 0" />
+      <inertia
+        ixx="0.001"
+        ixy="0"
+        ixz="0"
+        iyy="0.001"
+        iyz="0"
+        izz="0.001" />
+    </inertial>
+  </link>
+  <joint name="caster_joint" type="fixed">
+    <parent link="base_link"/>
+    <child link="caster_link"/>
+    <origin xyz="-0.245 0.0 0.032" rpy="${-M_PI/2} 0 0"/>
+    <axis xyz="0 0 1" />
   </joint>
   <link
@@ -252,5 +301,5 @@
     <origin
       xyz="-0.037385 0.1666 0"
-      rpy="1.5708 1.5708 0" />
+      rpy="-1.5708 1.5708 0" />
     <parent
       link="link_mast" />
@@ -369,5 +418,5 @@
     <axis
       xyz="0 0 1" />
-        <!-- 0.13 = 0.52/4-->
+    <!-- 0.13 = 0.52/4-->
     <limit effort="100" lower="0.0" upper="0.13" velocity="1.0"/>
   </joint>
@@ -582,5 +631,5 @@
     <origin
       xyz="0.0830000000000654 -0.0307500000000129 0"
-      rpy="-1.5707963267949 -6.34174103868745E-15 3.14159265358978" />
+      rpy="1.5708 4.2595E-14 2.6415E-15"/>
     <parent
       link="link_arm_l0" />
@@ -642,5 +691,5 @@
     <origin
       xyz="0 1.33 0"
-      rpy="1.5707963267949 -1.5707963267949 0" />
+      rpy="1.5707963267949 -1.5707963267949 3.1416" />
     <parent
       link="link_mast" />

Commit message: Mitski modified URDF merged to stretch_main.xacro

File: stretch_description/urdf/stretch_description.xacro (robot description, xacro)
@@ -4,6 +4,5 @@
   <!--<xacro:include filename="stretch_gripper_with_puller.xacro" />-->
   <!--<xacro:include filename="stretch_dry_erase_marker.xacro" />-->
-<!--  <xacro:include filename="stretch_main.xacro" />-->
-  <xacro:include filename="stretch_mitski.xacro" />
+  <xacro:include filename="stretch_main.xacro" />
   <xacro:include filename="stretch_aruco.xacro" />
   <xacro:include filename="stretch_d435i.xacro" />

File: stretch_description/urdf/stretch_main.xacro (robot description, xacro)
@@ -10,15 +10,15 @@
     <inertial>
       <origin
-        xyz="-0.109461304328163 -0.000741018909047708 0.0914915269429946"
-        rpy="0 0 0" />
-      <mass
-        value="1.0723782659782" />
-      <inertia
-        ixx="0.00310580907710135"
-        ixy="1.5182848191076E-06"
-        ixz="0.00041690466732394"
-        iyy="0.00433798719991832"
-        iyz="1.33487716258445E-05"
-        izz="0.0037204727467362" />
+        xyz="-0.11587 0.0019426 0.093621"
+        rpy="0 0 0" />
+      <mass
+        value="1.1912" />
+      <inertia
+        ixx="0.0034667"
+        ixy="-5.0568E-06"
+        ixz="0.00042861"
+        iyy="0.0052744"
+        iyz="-5.766E-05"
+        izz="0.0047945" />
     </inertial>
     <visual>
@@ -33,5 +33,5 @@
         name="">
         <color
-          rgba="0.792156862745098 0.819607843137255 0.933333333333333 1" />
+          rgba="0.79216 0.81961 0.93333 1" />
       </material>
     </visual>
@@ -50,15 +50,15 @@
     <inertial>
       <origin
-        xyz="1.25554620866719E-07 3.54748938447003E-07 0.0239581106165018"
-        rpy="0 0 0" />
-      <mass
-        value="0.01" />
-      <inertia
-        ixx="0.001"
+        xyz="1.1719E-11 2.0783E-11 0.037544"
+        rpy="0 0 0" />
+      <mass
+        value="0.0042721" />
+      <inertia
+        ixx="0"
         ixy="0"
         ixz="0"
-        iyy="0.001"
+        iyy="0"
         iyz="0"
-        izz="0.001" />
+        izz="0" />
     </inertial>
     <visual>
@@ -73,5 +73,5 @@
         name="">
         <color
-          rgba="0.792156862745098 0.819607843137255 0.933333333333333 1" />
+          rgba="0.79216 0.81961 0.93333 1" />
       </material>
     </visual>
@@ -90,6 +90,6 @@
     type="continuous">
     <origin
-      xyz="-0.00300000000000034 -0.15765 0.0508000000000004"
-      rpy="-1.57079632679489 -1.11022302462516E-16 7.28583859910277E-17" />
+      xyz="0 -0.17035 0.0508"
+      rpy="-1.5708 1.2717E-16 4.8006E-17" />
     <parent
       link="base_link" />
@@ -97,5 +97,5 @@
       link="link_right_wheel" />
     <axis
-      xyz="0 0 1" />
+      xyz="0 0 -1" />
     <dynamics damping="${joint_damping}" friction="${joint_friction}" spring_reference="${joint_spring_reference}" spring_stiffness="{joint_spring_stiffness}"/>
   </joint>
@@ -104,15 +104,15 @@
     <inertial>
       <origin
-        xyz="1.2555462092223E-07 -3.54748938502514E-07 -0.0239581106165035"
-        rpy="0 0 0" />
-      <mass
-        value="0.01" />
-      <inertia
-        ixx="0.001"
+        xyz="-2.0783E-11 -1.1719E-11 -0.037544"
+        rpy="0 0 0" />
+      <mass
+        value="0.0042721" />
+      <inertia
+        ixx="0"
         ixy="0"
         ixz="0"
-        iyy="0.001"
+        iyy="0"
         iyz="0"
-        izz="0.001" />
+        izz="0" />
     </inertial>
     <visual>
@@ -127,5 +127,5 @@
         name="">
         <color
-          rgba="0.792156862745098 0.819607843137255 0.933333333333333 1" />
+          rgba="0.79216 0.81961 0.93333 1" />
       </material>
     </visual>
@@ -144,6 +144,6 @@
     type="continuous">
     <origin
-      xyz="-0.00300000000001899 0.15765 0.0507999999999994"
-      rpy="-1.5707963267949 3.16227047920818E-31 7.88745438253713E-16" />
+      xyz="0 0.17035 0.0508"
+      rpy="-1.5708 2.6317E-16 -8.2057E-19" />
     <parent
       link="base_link" />
@@ -151,5 +151,5 @@
       link="link_left_wheel" />
     <axis
-      xyz="0 0 1" />
+      xyz="0 0 -1" />
     <dynamics damping="${joint_damping}" friction="${joint_friction}" spring_reference="${joint_spring_reference}" spring_stiffness="{joint_spring_stiffness}"/>
   </joint>
@@ -207,15 +207,15 @@
     <inertial>
       <origin
-        xyz="0.00755818572975822 0.773971284176834 0.00647313086620024"
-        rpy="0 0 0" />
-      <mass
-        value="0.749143203376401" />
-      <inertia
-        ixx="0.0709854511954588"
-        ixy="-0.00433428742758457"
-        ixz="-0.000186110788697573"
-        iyy="0.000437922053342648"
-        iyz="-0.00288788257713431"
-        izz="0.071104808501661" />
+        xyz="2.0817E-17 0.7075 -2.7756E-17"
+        rpy="0 0 0" />
+      <mass
+        value="1.8285" />
+      <inertia
+        ixx="0"
+        ixy="0"
+        ixz="0"
+        iyy="0"
+        iyz="0"
+        izz="0" />
     </inertial>
     <visual>
@@ -230,5 +230,5 @@
         name="">
         <color
-          rgba="0.792156862745098 0.819607843137255 0.933333333333333 1" />
+          rgba="0.79216 0.81961 0.93333 1" />
       </material>
     </visual>
@@ -247,6 +247,6 @@
     type="fixed">
     <origin
-      xyz="-0.07 0.134999999999998 0.0284000000000001"
-      rpy="1.5707963267949 0 0.00925318926571245" />
+      xyz="-0.067 0.135 0.0284"
+      rpy="1.5708 0 4.8006E-17" />
     <parent
       link="base_link" />
@@ -260,15 +260,15 @@
     <inertial>
       <origin
-        xyz="-0.0547636346252869 0.0380939689802074 0.00933159404448308"
-        rpy="0 0 0" />
-      <mass
-        value="0.444820831236007" />
-      <inertia
-        ixx="0.000567192946271367"
-        ixy="-0.00024607534789508"
-        ixz="-0.000128108442260574"
-        iyy="0.00127108364478659"
-        iyz="7.61916855070339E-06"
-        izz="0.00137296635099006" />
+        xyz="-0.031727 0.038403 0.013361"
+        rpy="0 0 0" />
+      <mass
+        value="0.27218" />
+      <inertia
+        ixx="0.00052571"
+        ixy="0.00014899"
+        ixz="-1.9258E-05"
+        iyy="0.00030679"
+        iyz="-6.2451E-06"
+        izz="0.00037324" />
     </inertial>
     <visual>
@@ -283,5 +283,5 @@
         name="">
         <color
-          rgba="0.792156862745098 0.819607843137255 0.933333333333333 1" />
+          rgba="0.79216 0.81961 0.93333 1" />
       </material>
     </visual>
@@ -300,6 +300,6 @@
     type="prismatic">
     <origin
-      xyz="-0.0369217062323472 0.165471199999996 -0.000341653286793524"
-      rpy="-1.57079632679552 1.5615431375292 -6.2942004366467E-13" />
+      xyz="-0.037385 0.1666 0"
+      rpy="-1.5708 1.5708 0" />
     <parent
       link="link_mast" />
@@ -307,5 +307,5 @@
       link="link_lift" />
     <axis
-	xyz="0 0 1" />
+      xyz="0 0 1" />
   <!-- for now: hand copied range_m: from lift: from ~/repos/stretch_fleet/stretch-re1-1001/stretch_re1_factory_params.yaml -->
   <!--<limit effort="100" lower="0.0" upper="1.095" velocity="1.0"/>-->
@@ -317,15 +317,15 @@
     <inertial>
       <origin
-        xyz="-1.61247276464493E-06 1.54715589201215E-06 -0.0953252706040035"
-        rpy="0 0 0" />
-      <mass
-        value="0.0676525455789735" />
-      <inertia
-        ixx="0.000122002023066796"
-        ixy="7.29593356230121E-13"
-        ixz="9.63170353371061E-09"
-        iyy="0.000122002023127152"
-        iyz="-9.24154949889042E-09"
-        izz="1.46043439809638E-12" />
+        xyz="-1.0146E-06 -1.9719E-05 -0.094738"
+        rpy="0 0 0" />
+      <mass
+        value="0.068095" />
+      <inertia
+        ixx="0.0001256"
+        ixy="-5.6914E-12"
+        ixz="6.0647E-09"
+        iyy="0.0001256"
+        iyz="1.1787E-07"
+        izz="1.1091E-10" />
     </inertial>
     <visual>
@@ -340,5 +340,5 @@
         name="">
         <color
-          rgba="0.792156862745098 0.819607843137255 0.933333333333333 1" />
+          rgba="0.79216 0.81961 0.93333 1" />
       </material>
     </visual>
@@ -357,6 +357,6 @@
     type="fixed">
     <origin
-      xyz="-0.25471 0 0"
-      rpy="1.5708 -3.1019E-16 -1.5708" />
+      xyz="-0.2547 0 0"
+      rpy="1.5708 2.4721E-15 -1.5708" />
     <parent
       link="link_lift" />
@@ -370,15 +370,15 @@
     <inertial>
       <origin
-        xyz="-3.34873468621488E-07 4.7411336306924E-07 -0.0974069598289041"
-        rpy="0 0 0" />
-      <mass
-        value="0.0626921047058405" />
-      <inertia
-        ixx="0.001"
-        ixy="0"
-        ixz="0"
-        iyy="0.001"
-        iyz="0"
-        izz="0.001" />
+        xyz="-5.13853606326845E-07 -1.99844969271112E-05 -0.0971104963726614"
+        rpy="0 0 0" />
+      <mass
+        value="0.0628927381893134" />
+      <inertia
+        ixx="0.000116972687184809"
+        ixy="-2.81979926511074E-12"
+        ixz="2.91222027599461E-09"
+        iyy="0.000116972577591313"
+        iyz="1.13260384471775E-07"
+        izz="1.09738504441915E-10" />
     </inertial>
     <visual>
@@ -411,5 +411,5 @@
     <origin
       xyz="0 0 0.013"
-      rpy="3.5742E-16 3.2123E-16 -2.4565E-16" />
+      rpy="7.68831233799385E-30 2.36716479416092E-30 2.29652732251143E-17" />
     <parent
       link="link_arm_l4" />
@@ -417,5 +417,5 @@
       link="link_arm_l3" />
     <axis
-	xyz="0 0 1" />
+      xyz="0 0 1" />
     <!-- 0.13 = 0.52/4-->
     <limit effort="100" lower="0.0" upper="0.13" velocity="1.0"/>
@@ -425,15 +425,15 @@
     <inertial>
       <origin
-        xyz="-3.31043560508615E-07 3.13422303999111E-07 -0.097255883541891"
-        rpy="0 0 0" />
-      <mass
-        value="0.0569074368576238" />
-      <inertia
-        ixx="0.001"
-        ixy="0"
-        ixz="0"
-        iyy="0.001"
-        iyz="0"
-        izz="0.001" />
+        xyz="-5.17421949435687E-07 -2.02045301450349E-05 -0.0968815475684904"
+        rpy="0 0 0" />
+      <mass
+        value="0.0571386353275368" />
+      <inertia
+        ixx="0.000107176369887422"
+        ixy="-2.57283392153217E-12"
+        ixz="2.65737742559071E-09"
+        iyy="0.000107176269488109"
+        iyz="1.0376649507793E-07"
+        izz="1.0053108970507E-10" />
     </inertial>
     <visual>
@@ -466,5 +466,5 @@
     <origin
       xyz="0 0 0.013"
-      rpy="2.91385731014123E-16 4.44300759504684E-17 3.25691080516352E-16" />
+      rpy="0 1.57655765344625E-30 -1.66533453693773E-16" />
     <parent
       link="link_arm_l3" />
@@ -472,5 +472,5 @@
       link="link_arm_l2" />
     <axis
-	xyz="0 0 1" />
+      xyz="0 0 1" />
     <!-- 0.13 = 0.52/4-->
     <limit effort="100" lower="0.0" upper="0.13" velocity="1.0"/>
@@ -480,15 +480,15 @@
     <inertial>
       <origin
-        xyz="-3.36876635420591E-07 3.05876091066803E-07 -0.0969117032232756"
-        rpy="0 0 0" />
-      <mass
-        value="0.0511763619538321" />
-      <inertia
-        ixx="0.001"
-        ixy="0"
-        ixz="0"
-        iyy="0.001"
-        iyz="0"
-        izz="0.001" />
+        xyz="-5.257E-07 -2.0482E-05 -0.096543"
+        rpy="0 0 0" />
+      <mass
+        value="0.051382" />
+      <inertia
+        ixx="9.7585E-05"
+        ixy="-2.3365E-12"
+        ixz="2.4191E-09"
+        iyy="9.7585E-05"
+        iyz="9.4252E-08"
+        izz="9.1094E-11" />
     </inertial>
     <visual>
@@ -503,5 +503,5 @@
         name="">
         <color
-          rgba="0.792156862745098 0.819607843137255 0.933333333333333 1" />
+          rgba="0.79216 0.81961 0.93333 1" />
       </material>
     </visual>
@@ -520,6 +520,6 @@
     type="prismatic">
     <origin
-      xyz="0 0 0.013"
-      rpy="7.41596560408007E-17 1.33876788296791E-16 -2.44545873596083E-16" />
+      xyz="0 0 0.0129999999999981"
+      rpy="-7.63746778746202E-30 -7.88860905221012E-31 1.11022302462516E-16" />
     <parent
       link="link_arm_l2" />
@@ -527,5 +527,5 @@
       link="link_arm_l1" />
     <axis
-	xyz="0 0 1" />
+      xyz="0 0 1" />
     <!-- 0.13 = 0.52/4-->
     <limit effort="100" lower="0.0" upper="0.13" velocity="1.0"/>
@@ -535,15 +535,15 @@
     <inertial>
       <origin
-        xyz="0.0230715049668191 -0.00195115833662818 -0.0360646347160285"
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
Commit message: Added DexWrist keyboard teleop and unified launch command for DexWrist config

File: stretch_description/urdf/stretch_description.xacro (robot description, xacro)
@@ -1,5 +1,6 @@
 <?xml version="1.0"?>
-<robot xmlns:xacro="http://www.ros.org/wiki/xacro" name="stretch">
-  <xacro:include filename="stretch_gripper.xacro" />
+<robot xmlns:xacro="http://www.ros.org/wiki/xacro" name="stretch_description">
+  <xacro:include filename="stretch_dex_wrist.xacro" />
+  <!--<xacro:include filename="stretch_gripper.xacro" /> -->
   <!--<xacro:include filename="stretch_gripper_with_puller.xacro" />-->
   <!--<xacro:include filename="stretch_dry_erase_marker.xacro" />-->
@@ -8,5 +9,4 @@
   <xacro:include filename="stretch_d435i.xacro" />
   <xacro:include filename="stretch_laser_range_finder.xacro" />
-  <xacro:include filename="stretch_base_imu.xacro" />
   <xacro:include filename="stretch_respeaker.xacro" />
 </robot>

File: stretch_gazebo/urdf/stretch_gazebo_dex_wrist.urdf.xacro (robot description, xacro)
@@ -8,5 +8,5 @@
   <xacro:include filename="$(find stretch_description)/urdf/stretch_laser_range_finder.xacro" />
   <xacro:include filename="$(find stretch_description)/urdf/stretch_respeaker.xacro" />
-  <xacro:include filename="$(find stretch_description)/urdf/stretch_gripper.xacro" />
+  <xacro:include filename="$(find stretch_description)/urdf/stretch_dex_wrist.xacro" />
   <gazebo>
     <plugin name="gazebo_ros_control" filename="libgazebo_ros_control.so">
@@ -487,53 +487,88 @@
     </joint>
   </transmission>
+  <!--Dex Wrist-->
+  <gazebo reference="link_wrist_yaw_bottom">
+      <mu1 value="100.0"/>
+      <mu2 value="200.0"/>
+      <kp value="10000000.0" />
+      <kd value="100.0" />
+      <material>Gazebo/Gray</material>
+      <minDepth>0.001</minDepth>
+  </gazebo>
+  <gazebo reference="link_wrist_pitch">
+      <mu1 value="100.0"/>
+      <mu2 value="200.0"/>
+      <kp value="10000000.0" />
+      <kd value="100.0" />
+      <material>Gazebo/Gray</material>
+      <minDepth>0.001</minDepth>
+  </gazebo>
+  <gazebo reference="link_wrist_roll">
+      <mu1 value="100.0"/>
+      <mu2 value="200.0"/>
+      <kp value="10000000.0" />
+      <kd value="100.0" />
+      <material>Gazebo/Gray</material>
+      <minDepth>0.001</minDepth>
+  </gazebo>
+  <gazebo reference="link_straight_gripper">
+      <mu1 value="100.0"/>
+      <mu2 value="200.0"/>
+      <kp value="10000000.0" />
+      <kd value="100.0" />
+      <material>Gazebo/Gray</material>
+      <minDepth>0.001</minDepth>
+  </gazebo>
+  <gazebo reference="link_gripper_finger_right">
+      <mu1 value="100.0"/>
+      <mu2 value="200.0"/>
+      <kp value="10000000.0" />
+      <kd value="100.0" />
+      <material>Gazebo/Gray</material>
+      <minDepth>0.001</minDepth>
+  </gazebo>
+  <gazebo reference="link_gripper_fingertip_right">
+      <mu1 value="100.0"/>
+      <mu2 value="200.0"/>
+      <kp value="10000000.0" />
+      <kd value="100.0" />
+      <material>Gazebo/Black</material>
+      <minDepth>0.001</minDepth>
+  </gazebo>
+  <gazebo reference="link_gripper_finger_left">
+      <mu1 value="100.0"/>
+      <mu2 value="200.0"/>
+      <kp value="10000000.0" />
+      <kd value="100.0" />
+      <material>Gazebo/Gray</material>
+      <minDepth>0.001</minDepth>
+  </gazebo>
+  <gazebo reference="link_gripper_fingertip_left">
+      <mu1 value="100.0"/>
+      <mu2 value="200.0"/>
+      <kp value="10000000.0" />
+      <kd value="100.0" />
+      <material>Gazebo/Black</material>
+      <minDepth>0.001</minDepth>
+  </gazebo>
+  <transmission name="trans_wrist_pitch">
+    <type>transmission_interface/SimpleTransmission</type>
+    <actuator name="motor_wrist_pitch">
+      <mechanicalReduction>1</mechanicalReduction>
+    </actuator>
+    <joint name="joint_wrist_pitch">
+      <hardwareInterface>hardware_interface/PositionJointInterface</hardwareInterface>
+    </joint>
+  </transmission>
+  <transmission name="trans_wrist_roll">
+    <type>transmission_interface/SimpleTransmission</type>
+    <actuator name="motor_wrist_roll">
+      <mechanicalReduction>1</mechanicalReduction>
+    </actuator>
+    <joint name="joint_wrist_roll">
+      <hardwareInterface>hardware_interface/PositionJointInterface</hardwareInterface>
+    </joint>
+  </transmission>
   <!-- Gripper -->
-  <gazebo reference="link_gripper_finger_left">
-      <mu1 value="100.0"/>
-      <mu2 value="200.0"/>
-      <kp value="10000000.0" />
-      <kd value="100.0" />
-      <material>Gazebo/Gray</material>
-      <minDepth>0.001</minDepth>
-  </gazebo>
-  <gazebo reference="link_gripper_finger_right">
-      <mu1 value="100.0"/>
-      <mu2 value="200.0"/>
-      <kp value="10000000.0" />
-      <kd value="100.0" />
-      <material>Gazebo/Gray</material>
-      <minDepth>0.001</minDepth>
-  </gazebo>
-  <gazebo reference="link_grasp_center">
-      <mu1 value="100.0"/>
-      <mu2 value="200.0"/>
-      <kp value="10000000.0" />
-      <kd value="100.0" />
-      <material>Gazebo/Gray</material>
-      <minDepth>0.001</minDepth>
-  </gazebo>
-  <gazebo reference="link_gripper_fingertip_left">
-      <mu1 value="100.0"/>
-      <mu2 value="200.0"/>
-      <kp value="10000000.0" />
-      <kd value="100.0" />
-      <material>Gazebo/Black</material>
-      <minDepth>0.001</minDepth>
-  </gazebo>
-  <gazebo reference="link_gripper_fingertip_right">
-      <mu1 value="100.0"/>
-      <mu2 value="200.0"/>
-      <kp value="10000000.0" />
-      <kd value="100.0" />
-      <material>Gazebo/Black</material>
-      <minDepth>0.001</minDepth>
-  </gazebo>
-  <gazebo reference="link_gripper">
-      <mu1 value="100.0"/>
-      <mu2 value="200.0"/>
-      <kp value="10000000.0" />
-      <kd value="100.0" />
-      <material>Gazebo/Gray</material>
-      <minDepth>0.001</minDepth>
-  </gazebo>
   <transmission name="trans_gripper_finger_left">
     <type>transmission_interface/SimpleTransmission</type>
@@ -553,4 +588,4 @@
       <hardwareInterface>hardware_interface/PositionJointInterface</hardwareInterface>
     </joint>
-</transmission>
+  </transmission>
 </robot>
