Commit message: Adds teleop kit support for dex wrist

File: stretch_description/urdf/stretch_base_imu.xacro (robot description, xacro)
@@ -8,12 +8,12 @@
         rpy="0 0 0" />
       <mass
-        value="0.00092" />
+        value="0.000901473198307758" />
       <inertia
-        ixx="3E-08"
-        ixy="0"
-        ixz="0"
-        iyy="5E-08"
-        iyz="0"
-        izz="8E-08" />
+        ixx="2.83324000746358E-08"
+        ixy="-2.10106175504755E-10"
+        ixz="1.86717014516205E-10"
+        iyy="5.35315990744214E-08"
+        iyz="9.31114208976591E-11"
+        izz="8.13221670783358E-08" />
     </inertial>
     <visual>

File: stretch_description/urdf/stretch_description_standard.xacro (robot description, xacro)
@@ -1,5 +1,6 @@
 <?xml version="1.0"?>
-<robot xmlns:xacro="http://www.ros.org/wiki/xacro" name="stretch">
+<robot xmlns:xacro="http://www.ros.org/wiki/xacro" name="stretch_description">
   <xacro:include filename="stretch_gripper.xacro" />
+  <!-- <xacro:include filename="stretch_dex_wrist.xacro" /> -->
   <!--<xacro:include filename="stretch_gripper_with_puller.xacro" />-->
   <!--<xacro:include filename="stretch_dry_erase_marker.xacro" />-->

File: stretch_description/urdf/stretch_gripper.xacro (robot description, xacro)
@@ -4,18 +4,17 @@
   <link
     name="link_gripper">
-    name="link_gripper">
-    <inertial>
-      <origin
-        xyz="-0.013687 0.015548 -0.035364"
-        rpy="0 0 0" />
-      <mass
-        value="0.175929" />
-      <inertia
-        ixx="0.000124"
-        ixy="3.7E-05"
-        ixz="5.7E-05"
-        iyy="0.000217"
-        iyz="1.1E-05"
-        izz="0.000221" />
+    <inertial>
+      <origin
+        xyz="-0.0170229132730066 0.0131410320934285 -0.0371614759484659"
+        rpy="0 0 0" />
+      <mass
+        value="0.101902711393094" />
+      <inertia
+        ixx="0.001"
+        ixy="0"
+        ixz="0"
+        iyy="0.001"
+        iyz="0"
+        izz="0.001" />
     </inertial>
     <visual>
@@ -62,15 +61,15 @@
     <inertial>
       <origin
-        xyz="0.094071 0.011377 0"
-        rpy="0 0 0" />
-      <mass
-        value="0.06" />
-      <inertia
-        ixx="1.1E-05"
-        ixy="3.6E-05"
-        ixz="0"
-        iyy="0.000214"
-        iyz="0"
-        izz="0.000224" />
+        xyz="0.0945047483510102 0.0124301080924361 -4.44089209850063E-16"
+        rpy="0 0 0" />
+      <mass
+        value="0.0476207785199474" />
+      <inertia
+        ixx="0.001"
+        ixy="0"
+        ixz="0"
+        iyy="0.001"
+        iyz="0"
+        izz="0.001" />
     </inertial>
     <visual>
@@ -116,15 +115,15 @@
     <inertial>
       <origin
-        xyz="0 0 0.008126"
-        rpy="0 0 0" />
-      <mass
-        value="0.003822" />
-      <inertia
-        ixx="0"
-        ixy="0"
-        ixz="0"
-        iyy="0"
-        iyz="0"
-        izz="1E-06" />
+        xyz="-3.16381381648689E-08 -2.91408530639359E-09 0.00812579670381812"
+        rpy="0 0 0" />
+      <mass
+        value="0.00382159917455729" />
+      <inertia
+        ixx="0.001"
+        ixy="0"
+        ixz="0"
+        iyy="0.001"
+        iyz="0"
+        izz="0.001" />
     </inertial>
     <visual>
@@ -169,15 +168,15 @@
     <inertial>
       <origin
-        xyz="-0.093921 -0.011351 0"
-        rpy="0 0 0" />
-      <mass
-        value="0.06" />
-      <inertia
-        ixx="1.1E-05"
-        ixy="3.6E-05"
-        ixz="0"
-        iyy="0.000213"
-        iyz="0"
-        izz="0.000223" />
+        xyz="-0.0945047483510099 -0.0124301080924345 0"
+        rpy="0 0 0" />
+      <mass
+        value="0.0476207785199481" />
+      <inertia
+        ixx="0.001"
+        ixy="0"
+        ixz="0"
+        iyy="0.001"
+        iyz="0"
+        izz="0.001" />
     </inertial>
     <visual>
@@ -223,15 +222,15 @@
     <inertial>
       <origin
-        xyz="0 0 0.008126"
-        rpy="0 0 0" />
-      <mass
-        value="0.003822" />
-      <inertia
-        ixx="0"
-        ixy="0"
-        ixz="0"
-        iyy="0"
-        iyz="0"
-        izz="1E-06" />
+        xyz="2.59386303963494E-08 6.70949018566347E-09 0.00812579516130402"
+        rpy="0 0 0" />
+      <mass
+        value="0.00382160037319545" />
+      <inertia
+        ixx="0.001"
+        ixy="0"
+        ixz="0"
+        iyy="0.001"
+        iyz="0"
+        izz="0.001" />
     </inertial>
     <visual>

File: stretch_description/urdf/stretch_gripper_with_puller.xacro (robot description, xacro)
@@ -6,15 +6,15 @@
     <inertial>
       <origin
-        xyz="-0.013687 0.015548 -0.035364"
-        rpy="0 0 0" />
-      <mass
-        value="0.175929" />
-      <inertia
-        ixx="0.000124"
-        ixy="3.7E-05"
-        ixz="5.7E-05"
-        iyy="0.000217"
-        iyz="1.1E-05"
-        izz="0.000221" />
+        xyz="-0.0170229132730066 0.0131410320934285 -0.0371614759484659"
+        rpy="0 0 0" />
+      <mass
+        value="0.101902711393094" />
+      <inertia
+        ixx="2.79241618017607E-05"
+        ixy="-1.10819247449605E-05"
+        ixz="-1.50343284036654E-05"
+        iyy="3.67945130513069E-05"
+        iyz="-4.33280448535579E-06"
+        izz="4.14524691955231E-05" />
     </inertial>
     <visual>
@@ -114,62 +114,8 @@
     <inertial>
       <origin
-        xyz="0.094071 0.011377 0"
-        rpy="0 0 0" />
-      <mass
-        value="0.06" />
-      <inertia
-        ixx="1.1E-05"
-        ixy="3.6E-05"
-        ixz="0"
-        iyy="0.000214"
-        iyz="0"
-        izz="0.000224" />
-    </inertial>
-    <visual>
-      <origin
-        xyz="0 0 0"
-        rpy="0 0 0" />
-      <geometry>
-        <mesh
-          filename="package://stretch_description/meshes/link_gripper_finger_left.STL" scale="${scale_finger_length} 1.0 1.0"/>
-      </geometry>
-      <material
-        name="">
-        <color
-          rgba="0.792156862745098 0.819607843137255 0.933333333333333 1" />
-      </material>
-    </visual>
-    <collision>
-      <origin
-        xyz="0 0 0"
-        rpy="0 0 0" />
-      <geometry>
-        <mesh
-          filename="package://stretch_description/meshes/link_gripper_finger_left.STL" scale="${scale_finger_length} 1.0 1.0"/>
-      </geometry>
-    </collision>
-  </link>
-  <joint
-    name="joint_gripper_finger_left"
-    type="revolute">
-    <origin
-      xyz="-0.047231 -0.010151 -0.04679"
-      rpy="2.1762E-15 0.5236 3.1416" />
-    <parent
-      link="link_gripper" />
-    <child
-      link="link_gripper_finger_left" />
-    <axis
-      xyz="0 0 1" />
-    <limit effort="100" lower="-0.6" upper="0.6" velocity="1.0"/>
-  </joint>
-  <link
-    name="link_gripper_fingertip_left">
-    <inertial>
-      <origin
-        xyz="0 0 0.008126"
-        rpy="0 0 0" />
-      <mass
-        value="0.003822" />
+        xyz="0.0945047483510102 0.0124301080924361 -4.44089209850063E-16"
+        rpy="0 0 0" />
+      <mass
+        value="0.0476207785199474" />
       <inertia
         ixx="0"
@@ -178,93 +124,40 @@
         iyy="0"
         iyz="0"
-        izz="1E-06" />
-    </inertial>
-    <visual>
-      <origin
-        xyz="0 0 0"
-        rpy="0 0 0" />
-      <geometry>
-        <mesh
-          filename="package://stretch_description/meshes/link_gripper_fingertip_left.STL" />
-      </geometry>
-      <material
-        name="">
-        <color
-          rgba="0.250980392156863 0.250980392156863 0.250980392156863 1" />
-      </material>
-    </visual>
-    <collision>
-      <origin
-        xyz="0 0 0"
-        rpy="0 0 0" />
-      <geometry>
-        <mesh
-          filename="package://stretch_description/meshes/link_gripper_fingertip_left.STL" />
-      </geometry>
-    </collision>
-  </link>
-  <joint
-    name="joint_gripper_fingertip_left"
-    type="fixed">
-    <origin
-      xyz="${scale_finger_length * 0.19011} 0.014912 0"
-      rpy="-1.5708 -4.774E-15 -2.5545" />
-    <parent
+        izz="0" />
+    </inertial>
+    <visual>
+      <origin
+        xyz="0 0 0"
+        rpy="0 0 0" />
+      <geometry>
+        <mesh
+          filename="package://stretch_description/meshes/link_gripper_finger_left.STL" scale="${scale_finger_length} 1.0 1.0"/>
+      </geometry>
+      <material
+        name="">
+        <color
+          rgba="0.792156862745098 0.819607843137255 0.933333333333333 1" />
+      </material>
+    </visual>
+    <collision>
+      <origin
+        xyz="0 0 0"
+        rpy="0 0 0" />
+      <geometry>
+        <mesh
+          filename="package://stretch_description/meshes/link_gripper_finger_left.STL" scale="${scale_finger_length} 1.0 1.0"/>
+      </geometry>
+    </collision>
+  </link>
+  <joint
+    name="joint_gripper_finger_left"
+    type="revolute">
+    <origin
+      xyz="-0.047231 -0.010151 -0.04679"
+      rpy="2.1762E-15 0.5236 3.1416" />
+    <parent
+      link="link_gripper" />
+    <child
       link="link_gripper_finger_left" />
-    <child
-      link="link_gripper_fingertip_left" />
-    <axis
-      xyz="0 0 0" />
-  </joint>
-  <link
-    name="link_gripper_finger_right">
-    <inertial>
-      <origin
-        xyz="-0.093921 -0.011351 0"
-        rpy="0 0 0" />
-      <mass
-        value="0.06" />
-      <inertia
-        ixx="1.1E-05"
-        ixy="3.6E-05"
-        ixz="0"
-        iyy="0.000213"
-        iyz="0"
-        izz="0.000223" />
-    </inertial>
-    <visual>
-      <origin
-        xyz="0 0 0"
-        rpy="0 0 0" />
-      <geometry>
-        <mesh
-          filename="package://stretch_description/meshes/link_gripper_finger_right.STL" scale="${scale_finger_length} 1.0 1.0"/>
-      </geometry>
-      <material
-        name="">
-        <color
-          rgba="0.792156862745098 0.819607843137255 0.933333333333333 1" />
-      </material>
-    </visual>
-    <collision>
-      <origin
-        xyz="0 0 0"
-        rpy="0 0 0" />
-      <geometry>
-        <mesh
-          filename="package://stretch_description/meshes/link_gripper_finger_right.STL" scale="${scale_finger_length} 1.0 1.0"/>
-      </geometry>
-    </collision>
-  </link>
-  <joint
-    name="joint_gripper_finger_right"
-    type="revolute">
-    <origin
-      xyz="-0.047231 0.010049 -0.04679"
-      rpy="3.1416 -0.5236 1.2943E-15" />
-    <parent
-      link="link_gripper" />
-    <child
-      link="link_gripper_finger_right" />
     <axis
       xyz="0 0 1" />
@@ -272,11 +165,11 @@
   </joint>
   <link
-    name="link_gripper_fingertip_right">
-    <inertial>
-      <origin
-        xyz="0 0 0.008126"
-        rpy="0 0 0" />
-      <mass
-        value="0.003822" />
+    name="link_gripper_fingertip_left">
+    <inertial>
+      <origin
+        xyz="-3.16381381648689E-08 -2.91408530639359E-09 0.00812579670381812"
+        rpy="0 0 0" />
+      <mass
+        value="0.00382159917455729" />
       <inertia
         ixx="0"
@@ -285,5 +178,112 @@
         iyy="0"
         iyz="0"
-        izz="1E-06" />
+        izz="0" />
+    </inertial>
+    <visual>
+      <origin
+        xyz="0 0 0"
+        rpy="0 0 0" />
+      <geometry>
+        <mesh
+          filename="package://stretch_description/meshes/link_gripper_fingertip_left.STL" />
+      </geometry>
+      <material
+        name="">
+        <color
+          rgba="0.250980392156863 0.250980392156863 0.250980392156863 1" />
+      </material>
+    </visual>
+    <collision>
+      <origin
+        xyz="0 0 0"
+        rpy="0 0 0" />
+      <geometry>
+        <mesh
+          filename="package://stretch_description/meshes/link_gripper_fingertip_left.STL" />
+      </geometry>
+    </collision>
+  </link>
+  <joint
+    name="joint_gripper_fingertip_left"
+    type="fixed">
+    <origin
+      xyz="${scale_finger_length * 0.19011} 0.014912 0"
+      rpy="-1.5708 -4.774E-15 -2.5545" />
+    <parent
+      link="link_gripper_finger_left" />
+    <child
+      link="link_gripper_fingertip_left" />
+    <axis
+      xyz="0 0 0" />
+  </joint>
+  <link
+    name="link_gripper_finger_right">
+    <inertial>
+      <origin
+        xyz="-0.0945047483510099 -0.0124301080924345 0"
+        rpy="0 0 0" />
+      <mass
+        value="0.0476207785199481" />
+      <inertia
+        ixx="0"
+        ixy="0"
+        ixz="0"
+        iyy="0"
+        iyz="0"
+        izz="0" />
+    </inertial>
+    <visual>
+      <origin
+        xyz="0 0 0"
+        rpy="0 0 0" />
+      <geometry>
+        <mesh
+          filename="package://stretch_description/meshes/link_gripper_finger_right.STL" scale="${scale_finger_length} 1.0 1.0"/>
+      </geometry>
+      <material
+        name="">
+        <color
+          rgba="0.792156862745098 0.819607843137255 0.933333333333333 1" />
+      </material>
+    </visual>
+    <collision>
+      <origin
+        xyz="0 0 0"
+        rpy="0 0 0" />
+      <geometry>
+        <mesh
+          filename="package://stretch_description/meshes/link_gripper_finger_right.STL" scale="${scale_finger_length} 1.0 1.0"/>
+      </geometry>
+    </collision>
+  </link>
+  <joint
+    name="joint_gripper_finger_right"
+    type="revolute">
+    <origin
+      xyz="-0.047231 0.010049 -0.04679"
+      rpy="3.1416 -0.5236 1.2943E-15" />
+    <parent
+      link="link_gripper" />
+    <child
+      link="link_gripper_finger_right" />
+    <axis
+      xyz="0 0 1" />
+    <limit effort="100" lower="-0.6" upper="0.6" velocity="1.0"/>
+  </joint>
+  <link
+    name="link_gripper_fingertip_right">
+    <inertial>
+      <origin
+        xyz="2.59386303963494E-08 6.70949018566347E-09 0.00812579516130402"
+        rpy="0 0 0" />
+      <mass
+        value="0.00382160037319545" />
+      <inertia
+        ixx="0"
+        ixy="0"
+        ixz="0"
+        iyy="0"
+        iyz="0"
+        izz="0" />
     </inertial>
     <visual>

File: stretch_description/urdf/stretch_laser_range_finder.xacro (robot description, xacro)
@@ -5,15 +5,15 @@
     <inertial>
       <origin
-        xyz="0.011979 -0.000523 -0.01998"
+        xyz="0 0 -0.000755956127492408"
         rpy="0 0 0" />
       <mass
-        value="0.216007" />
+        value="0.0749979022894495" />
       <inertia
-        ixx="9.5E-05"
-        ixy="2E-06"
-        ixz="-1.9E-05"
-        iyy="0.000184"
-        iyz="-1E-06"
-        izz="0.000216" />
+        ixx="0"
+        ixy="0"
+        ixz="0"
+        iyy="0"
+        iyz="0"
+        izz="0" />
     </inertial>
     <visual>
