Commit message: Adds teleop kit support for dex wrist

File: stretch_description/urdf/stretch_main.xacro (robot description, xacro)
@@ -10,15 +10,15 @@
     <inertial>
       <origin
-        xyz="-0.087526 -0.001626 0.081009"
-        rpy="0 0 0" />
-      <mass
-        value="17.384389" />
-      <inertia
-        ixx="0.160002"
-        ixy="0.006758"
-        ixz="0.004621"
-        iyy="0.138068"
-        iyz="0.002208"
-        izz="0.228992" />
+        xyz="-0.11587 0.0019426 0.093621"
+        rpy="0 0 0" />
+      <mass
+        value="1.1912" />
+      <inertia
+        ixx="0.0034667"
+        ixy="-5.0568E-06"
+        ixz="0.00042861"
+        iyy="0.0052744"
+        iyz="-5.766E-05"
+        izz="0.0047945" />
     </inertial>
     <visual>
@@ -50,15 +50,15 @@
     <inertial>
       <origin
-        xyz="0 0 0.02765"
-        rpy="0 0 0" />
-      <mass
-        value="0.20773" />
-      <inertia
-        ixx="5.4E-05"
-        ixy="0"
-        ixz="0"
-        iyy="5.4E-05"
-        iyz="0"
-        izz="5.1E-05" />
+        xyz="1.1719E-11 2.0783E-11 0.037544"
+        rpy="0 0 0" />
+      <mass
+        value="0.0042721" />
+      <inertia
+        ixx="0.001"
+        ixy="0"
+        ixz="0"
+        iyy="0.001"
+        iyz="0"
+        izz="0.001" />
     </inertial>
     <visual>
@@ -104,15 +104,15 @@
     <inertial>
       <origin
-        xyz="0 0 -0.02765"
-        rpy="0 0 0" />
-      <mass
-        value="0.20773" />
-      <inertia
-        ixx="5.4E-05"
-        ixy="0"
-        ixz="0"
-        iyy="5.4E-05"
-        iyz="0"
-        izz="5.1E-05" />
+        xyz="-2.0783E-11 -1.1719E-11 -0.037544"
+        rpy="0 0 0" />
+      <mass
+        value="0.0042721" />
+      <inertia
+        ixx="0.001"
+        ixy="0"
+        ixz="0"
+        iyy="0.001"
+        iyz="0"
+        izz="0.001" />
     </inertial>
     <visual>
@@ -207,15 +207,15 @@
     <inertial>
       <origin
-        xyz="0.000337 0.722201 0.002652"
-        rpy="0 0 0" />
-      <mass
-        value="1.764017" />
-      <inertia
-        ixx="0.291286"
-        ixy="0.004149"
-        ixz="-0.000174"
-        iyy="0.001226"
-        iyz="0.000354"
-        izz="0.291429" />
+        xyz="2.0817E-17 0.7075 -2.7756E-17"
+        rpy="0 0 0" />
+      <mass
+        value="1.8285" />
+      <inertia
+        ixx="0.0709854511954588"
+        ixy="-0.00433428742758457"
+        ixz="-0.000186110788697573"
+        iyy="0.000437922053342648"
+        iyz="-0.00288788257713431"
+        izz="0.071104808501661" />
     </inertial>
     <visual>
@@ -260,15 +260,15 @@
     <inertial>
       <origin
-        xyz="-0.020369 0.03438 0.02236"
-        rpy="0 0 0" />
-      <mass
-        value="1.987167" />
-      <inertia
-        ixx="0.006518"
-        ixy="-0.001539"
-        ixz="0.000371"
-        iyy="0.004464"
-        iyz="0.000392"
-        izz="0.008092" />
+        xyz="-0.031727 0.038403 0.013361"
+        rpy="0 0 0" />
+      <mass
+        value="0.27218" />
+      <inertia
+        ixx="0.00052571"
+        ixy="0.00014899"
+        ixz="-1.9258E-05"
+        iyy="0.00030679"
+        iyz="-6.2451E-06"
+        izz="0.00037324" />
     </inertial>
     <visual>
@@ -308,5 +308,5 @@
     <axis
       xyz="0 0 1" />
-  <!-- for now: hand copied range_m: from lift: from ~/repos/stretch_fleet/stretch-re1-1001/stretch_re1_factory_params.yaml -->
+  <!-- for now hand copied range_m from lift from ~/repos/stretch_fleet/stretch-re1-1001/stretch_re1_factory_params.yaml -->
   <!--<limit effort="100" lower="0.0" upper="1.095" velocity="1.0"/>-->
   <!-- copied value did not reach the top of mesh model with GUI sliders and RViz -->
@@ -317,15 +317,15 @@
     <inertial>
       <origin
-        xyz="-0.000168 -0.000254 -0.125235"
-        rpy="0 0 0" />
-      <mass
-        value="0.235626" />
-      <inertia
-        ixx="0.001518"
-        ixy="-1E-06"
-        ixz="3E-06"
-        iyy="0.001519"
-        iyz="3E-06"
-        izz="0.000176" />
+        xyz="-1.0146E-06 -1.9719E-05 -0.094738"
+        rpy="0 0 0" />
+      <mass
+        value="0.068095" />
+      <inertia
+        ixx="0.0001256"
+        ixy="-5.6914E-12"
+        ixz="6.0647E-09"
+        iyy="0.0001256"
+        iyz="1.1787E-07"
+        izz="1.1091E-10" />
     </inertial>
     <visual>
@@ -370,15 +370,15 @@
     <inertial>
       <origin
-        xyz="-1E-06 -0.000146 -0.11908"
-        rpy="0 0 0" />
-      <mass
-        value="0.146817" />
-      <inertia
-        ixx="0.001081"
-        ixy="0"
-        ixz="0"
-        iyy="0.001081"
-        iyz="-1E-06"
-        izz="7.7E-05" />
+        xyz="-5.13853606326845E-07 -1.99844969271112E-05 -0.0971104963726614"
+        rpy="0 0 0" />
+      <mass
+        value="0.0628927381893134" />
+      <inertia
+        ixx="0.001"
+        ixy="0"
+        ixz="0"
+        iyy="0.001"
+        iyz="0"
+        izz="0.001" />
     </inertial>
     <visual>
@@ -425,15 +425,15 @@
     <inertial>
       <origin
-        xyz="0 -7.1E-05 -0.115635"
-        rpy="0 0 0" />
-      <mass
-        value="0.130565" />
-      <inertia
-        ixx="0.000943"
-        ixy="0"
-        ixz="0"
-        iyy="0.000943"
-        iyz="0"
-        izz="5.7E-05" />
+        xyz="-5.17421949435687E-07 -2.02045301450349E-05 -0.0968815475684904"
+        rpy="0 0 0" />
+      <mass
+        value="0.0571386353275368" />
+      <inertia
+        ixx="0.001"
+        ixy="0"
+        ixz="0"
+        iyy="0.001"
+        iyz="0"
+        izz="0.001" />
     </inertial>
     <visual>
@@ -480,15 +480,15 @@
     <inertial>
       <origin
-        xyz="-1E-06 -0.000121 -0.113457"
-        rpy="0 0 0" />
-      <mass
-        value="0.113658" />
-      <inertia
-        ixx="0.0008"
-        ixy="0"
-        ixz="0"
-        iyy="0.0008"
-        iyz="0"
-        izz="4E-05" />
+        xyz="-5.257E-07 -2.0482E-05 -0.096543"
+        rpy="0 0 0" />
+      <mass
+        value="0.051382" />
+      <inertia
+        ixx="0.001"
+        ixy="0"
+        ixz="0"
+        iyy="0.001"
+        iyz="0"
+        izz="0.001" />
     </inertial>
     <visual>
@@ -535,15 +535,15 @@
     <inertial>
       <origin
-        xyz="0.033681 -0.000847 -0.031723"
-        rpy="0 0 0" />
-      <mass
-        value="0.427734" />
-      <inertia
-        ixx="0.001689"
-        ixy="-2.8E-05"
-        ixz="0.000483"
-        iyy="0.002107"
-        iyz="-1.1E-05"
-        izz="0.000571" />
+        xyz="0.0270582141286185 -0.00189876414654466 -0.0377809018481181"
+        rpy="0 0 0" />
+      <mass
+        value="0.085003260946398" />
+      <inertia
+        ixx="0.001"
+        ixy="0"
+        ixz="0"
+        iyy="0.001"
+        iyz="0"
+        izz="0.001" />
     </inertial>
     <visual>
@@ -590,15 +590,15 @@
     <inertial>
       <origin
-        xyz="0 -3.9E-05 -0.016495"
-        rpy="0 0 0" />
-      <mass
-        value="0.054422" />
-      <inertia
-        ixx="9E-06"
-        ixy="0"
-        ixz="0"
-        iyy="9E-06"
-        iyz="0"
-        izz="7E-06" />
+        xyz="2.20122392535771E-11 2.9317167880849E-05 -0.018966592644729"
+        rpy="0 0 0" />
+      <mass
+        value="0.0404746907425003" />
+      <inertia
+        ixx="0.001"
+        ixy="0"
+        ixz="0"
+        iyy="0.001"
+        iyz="0"
+        izz="0.001" />
     </inertial>
     <visual>
@@ -639,7 +639,7 @@
       xyz="0 0 -1" />
     <!--
-      stowed to front ~225 deg: 3.15159 x 1.25 = 3.9395
+      stowed to front ~225 deg, 3.15159 x 1.25 = 3.9395
       using 4.0
-      stowed to back ~100 deg:  100 / 180 x 3.14159 = 1.7453
+      stowed to back ~100 deg, 100 / 180 x 3.14159 = 1.7453
       using -1.75
     -->
@@ -650,15 +650,15 @@
     <inertial>
       <origin
-        xyz="0.047462 0.04451 0.016376"
-        rpy="0 0 0" />
-      <mass
-        value="0.681871" />
-      <inertia
-        ixx="0.001023"
-        ixy="0.000641"
-        ixz="6.6E-05"
-        iyy="0.002097"
-        iyz="6.5E-05"
-        izz="0.00281" />
+        xyz="0.0406850995527703 0.0396956343318414 0.0226500246461012"
+        rpy="0 0 0" />
+      <mass
+        value="0.133027236718691" />
+      <inertia
+        ixx="0.001"
+        ixy="0"
+        ixz="0"
+        iyy="0.001"
+        iyz="0"
+        izz="0.001" />
     </inertial>
     <visual>
@@ -703,15 +703,15 @@
     <inertial>
       <origin
-        xyz="-0.000422 0.013934 -0.0161"
-        rpy="0 0 0" />
-      <mass
-        value="0.062462" />
-      <inertia
-        ixx="4.1E-05"
-        ixy="-1E-06"
-        ixz="1E-06"
-        iyy="3.2E-05"
-        iyz="-1.5E-05"
-        izz="2.2E-05" />
+        xyz="-0.000326562615178591 0.00850012613776489 0.000130487222982367"
+        rpy="0 0 0" />
+      <mass
+        value="0.0273764496535409" />
+      <inertia
+        ixx="0.001"
+        ixy="0"
+        ixz="0"
+        iyy="0.001"
+        iyz="0"
+        izz="0.001" />
     </inertial>
     <visual>
@@ -758,15 +758,15 @@
     <inertial>
       <origin
-        xyz="0.003907 -0.02418 0.030154"
-        rpy="0 0 0" />
-      <mass
-        value="0.283548" />
-      <inertia
-        ixx="0.000316"
-        ixy="-6E-06"
-        ixz="1E-06"
-        iyy="0.000143"
-        iyz="-2E-06"
-        izz="0.00031" />
+        xyz="0.00704566394917504 -0.0212256210929691 0.0302058990060359"
+        rpy="0 0 0" />
+      <mass
+        value="0.090217113313934" />
+      <inertia
+        ixx="0.001"
+        ixy="0"
+        ixz="0"
+        iyy="0.001"
+        iyz="0"
+        izz="0.001" />
     </inertial>
     <visual>

File: stretch_description/urdf/stretch_respeaker.xacro (robot description, xacro)
@@ -5,15 +5,15 @@
     <inertial>
       <origin
-        xyz="-0.001594 -0.001282 -0.008098"
+        xyz="-0.003809 -0.0023075 -0.012854"
         rpy="0 0 0" />
       <mass
-        value="0.025175" />
+        value="0.015643" />
       <inertia
-        ixx="1E-05"
-        ixy="2E-06"
-        ixz="1E-06"
-        iyy="1.2E-05"
-        iyz="0"
-        izz="1.5E-05" />
+        ixx="1.0075E-06"
+        ixy="-5.4396E-08"
+        ixz="-2.8652E-07"
+        iyy="1.0569E-06"
+        iyz="-1.8463E-07"
+        izz="1.1947E-07" />
     </inertial>
     <visual>

File: stretch_gazebo/urdf/stretch_gazebo_dex_wrist.urdf.xacro (robot description, xacro)
@@ -9,4 +9,5 @@
   <xacro:include filename="$(find stretch_gazebo)/urdf/stretch_respeaker.xacro" />
   <xacro:include filename="$(find stretch_gazebo)/urdf/stretch_dex_wrist.xacro" />
+  <!-- <xacro:include filename="$(find stretch_gazebo)/urdf/stretch_teleop_kit_dex_wrist.xacro" />  -->
   <gazebo>
     <plugin name="gazebo_ros_control" filename="libgazebo_ros_control.so">
@@ -60,4 +61,77 @@
 		</transmission>
   <!-- Sensors -->
+<!--Teleop Cameras-->
+  <gazebo reference="link_gripper_teleop_camera">
+    <sensor type="camera" name="gripper_teleop_camera">
+      <update_rate>30.0</update_rate>
+      <camera name="gripper_teleop_camera">
+        <horizontal_fov>2.26</horizontal_fov>
+        <image>
+          <width>640</width>
+          <height>480</height>
+          <format>R8G8B8</format>
+        </image>
+        <clip>
+          <near>0.02</near>
+          <far>300</far>
+        </clip>
+        <noise>
+          <type>gaussian</type>
+          <mean>0.0</mean>
+          <stddev>0.007</stddev>
+        </noise>
+      </camera>
+      <plugin name="camera_controller" filename="libgazebo_ros_camera.so">
+        <alwaysOn>true</alwaysOn>
+        <updateRate>0.0</updateRate>
+        <cameraName>teleop/gripper_camera</cameraName>
+        <imageTopicName>image_raw</imageTopicName>
+        <cameraInfoTopicName>camera_info</cameraInfoTopicName>
+        <frameName>camera_link</frameName>
+        <hackBaseline>0.07</hackBaseline>
+        <distortionK1>0.0</distortionK1>
+        <distortionK2>0.0</distortionK2>
+        <distortionK3>0.0</distortionK3>
+        <distortionT1>0.0</distortionT1>
+        <distortionT2>0.0</distortionT2>
+      </plugin>
+    </sensor>
+  </gazebo>
+  <gazebo reference="link_head_teleop_camera">
+    <sensor type="camera" name="head_teleop_camera">
+      <update_rate>30.0</update_rate>
+      <camera name="head_teleop_camera">
+        <horizontal_fov>2.26</horizontal_fov>
+        <image>
+          <width>640</width>
+          <height>480</height>
+          <format>R8G8B8</format>
+        </image>
+        <clip>
+          <near>0.02</near>
+          <far>300</far>
+        </clip>
+        <noise>
+          <type>gaussian</type>
+          <mean>0.0</mean>
+          <stddev>0.007</stddev>
+        </noise>
+      </camera>
+      <plugin name="camera_controller" filename="libgazebo_ros_camera.so">
+        <alwaysOn>true</alwaysOn>
+        <updateRate>0.0</updateRate>
+        <cameraName>teleop/head_camera</cameraName>
+        <imageTopicName>image_raw</imageTopicName>
+        <cameraInfoTopicName>camera_info</cameraInfoTopicName>
+        <frameName>camera_link</frameName>
+        <hackBaseline>0.07</hackBaseline>
+        <distortionK1>0.0</distortionK1>
+        <distortionK2>0.0</distortionK2>
+        <distortionK3>0.0</distortionK3>
+        <distortionT1>0.0</distortionT1>
+        <distortionT2>0.0</distortionT2>
+      </plugin>
+    </sensor>
+  </gazebo>
   <!-- Realsense D435i -->
   <gazebo reference="camera_color_frame">

File: stretch_gazebo/urdf/stretch_gazebo_standard_gripper.urdf.xacro (robot description, xacro)
@@ -9,4 +9,5 @@
   <xacro:include filename="$(find stretch_gazebo)/urdf/stretch_respeaker.xacro" />
   <xacro:include filename="$(find stretch_gazebo)/urdf/stretch_gripper.xacro" />
+  <xacro:include filename="$(find stretch_gazebo)/urdf/stretch_teleop_kit_standard_gripper.xacro" />
   <gazebo>
     <plugin name="gazebo_ros_control" filename="libgazebo_ros_control.so">
