Commit message: new mass data ready and tested

File: stretch_description/batch/mitski/urdf/stretch_gripper.xacro (robot description, xacro)
@@ -4,17 +4,18 @@
   <link
     name="link_gripper">
-    <inertial>
-      <origin
-        xyz="-0.0170229132730066 0.0131410320934285 -0.0371614759484659"
-        rpy="0 0 0" />
-      <mass
-        value="0.101902711393094" />
-      <inertia
-        ixx="0.001"
-        ixy="0"
-        ixz="0"
-        iyy="0.001"
-        iyz="0"
-        izz="0.001" />
+    name="link_gripper">
+    <inertial>
+      <origin
+        xyz="-0.013687 0.015548 -0.035364"
+        rpy="0 0 0" />
+      <mass
+        value="0.175929" />
+      <inertia
+        ixx="0.000124"
+        ixy="3.7E-05"
+        ixz="5.7E-05"
+        iyy="0.000217"
+        iyz="1.1E-05"
+        izz="0.000221" />
     </inertial>
     <visual>
@@ -61,15 +62,15 @@
     <inertial>
       <origin
-        xyz="0.0945047483510102 0.0124301080924361 -4.44089209850063E-16"
-        rpy="0 0 0" />
-      <mass
-        value="0.0476207785199474" />
-      <inertia
-        ixx="0.001"
-        ixy="0"
-        ixz="0"
-        iyy="0.001"
-        iyz="0"
-        izz="0.001" />
+        xyz="0.094071 0.011377 0"
+        rpy="0 0 0" />
+      <mass
+        value="0.06" />
+      <inertia
+        ixx="1.1E-05"
+        ixy="3.6E-05"
+        ixz="0"
+        iyy="0.000214"
+        iyz="0"
+        izz="0.000224" />
     </inertial>
     <visual>
@@ -115,15 +116,15 @@
     <inertial>
       <origin
-        xyz="-3.16381381648689E-08 -2.91408530639359E-09 0.00812579670381812"
-        rpy="0 0 0" />
-      <mass
-        value="0.00382159917455729" />
-      <inertia
-        ixx="0.001"
+        xyz="0 0 0.008126"
+        rpy="0 0 0" />
+      <mass
+        value="0.003822" />
+      <inertia
+        ixx="0"
         ixy="0"
         ixz="0"
-        iyy="0.001"
-        iyz="0"
-        izz="0.001" />
+        iyy="0"
+        iyz="0"
+        izz="1E-06" />
     </inertial>
     <visual>
@@ -168,15 +169,15 @@
     <inertial>
       <origin
-        xyz="-0.0945047483510099 -0.0124301080924345 0"
-        rpy="0 0 0" />
-      <mass
-        value="0.0476207785199481" />
-      <inertia
-        ixx="0.001"
-        ixy="0"
-        ixz="0"
-        iyy="0.001"
-        iyz="0"
-        izz="0.001" />
+        xyz="-0.093921 -0.011351 0"
+        rpy="0 0 0" />
+      <mass
+        value="0.06" />
+      <inertia
+        ixx="1.1E-05"
+        ixy="3.6E-05"
+        ixz="0"
+        iyy="0.000213"
+        iyz="0"
+        izz="0.000223" />
     </inertial>
     <visual>
@@ -222,15 +223,15 @@
     <inertial>
       <origin
-        xyz="2.59386303963494E-08 6.70949018566347E-09 0.00812579516130402"
-        rpy="0 0 0" />
-      <mass
-        value="0.00382160037319545" />
-      <inertia
-        ixx="0.001"
+        xyz="0 0 0.008126"
+        rpy="0 0 0" />
+      <mass
+        value="0.003822" />
+      <inertia
+        ixx="0"
         ixy="0"
         ixz="0"
-        iyy="0.001"
-        iyz="0"
-        izz="0.001" />
+        iyy="0"
+        iyz="0"
+        izz="1E-06" />
     </inertial>
     <visual>

File: stretch_description/batch/mitski/urdf/stretch_gripper_with_puller.xacro (robot description, xacro)
@@ -6,15 +6,15 @@
     <inertial>
       <origin
-        xyz="-0.0170229132730066 0.0131410320934285 -0.0371614759484659"
-        rpy="0 0 0" />
-      <mass
-        value="0.101902711393094" />
-      <inertia
-        ixx="2.79241618017607E-05"
-        ixy="-1.10819247449605E-05"
-        ixz="-1.50343284036654E-05"
-        iyy="3.67945130513069E-05"
-        iyz="-4.33280448535579E-06"
-        izz="4.14524691955231E-05" />
+        xyz="-0.013687 0.015548 -0.035364"
+        rpy="0 0 0" />
+      <mass
+        value="0.175929" />
+      <inertia
+        ixx="0.000124"
+        ixy="3.7E-05"
+        ixz="5.7E-05"
+        iyy="0.000217"
+        iyz="1.1E-05"
+        izz="0.000221" />
     </inertial>
     <visual>
@@ -114,8 +114,62 @@
     <inertial>
       <origin
-        xyz="0.0945047483510102 0.0124301080924361 -4.44089209850063E-16"
-        rpy="0 0 0" />
-      <mass
-        value="0.0476207785199474" />
+        xyz="0.094071 0.011377 0"
+        rpy="0 0 0" />
+      <mass
+        value="0.06" />
+      <inertia
+        ixx="1.1E-05"
+        ixy="3.6E-05"
+        ixz="0"
+        iyy="0.000214"
+        iyz="0"
+        izz="0.000224" />
+    </inertial>
+    <visual>
+      <origin
+        xyz="0 0 0"
+        rpy="0 0 0" />
+      <geometry>
+        <mesh
+          filename="package://stretch_description/meshes/link_gripper_finger_left.STL" scale="${scale_finger_length} 1.0 1.0"/>
+      </geometry>
+      <material
+        name="">
+        <color
+          rgba="0.792156862745098 0.819607843137255 0.933333333333333 1" />
+      </material>
+    </visual>
+    <collision>
+      <origin
+        xyz="0 0 0"
+        rpy="0 0 0" />
+      <geometry>
+        <mesh
+          filename="package://stretch_description/meshes/link_gripper_finger_left.STL" scale="${scale_finger_length} 1.0 1.0"/>
+      </geometry>
+    </collision>
+  </link>
+  <joint
+    name="joint_gripper_finger_left"
+    type="revolute">
+    <origin
+      xyz="-0.047231 -0.010151 -0.04679"
+      rpy="2.1762E-15 0.5236 3.1416" />
+    <parent
+      link="link_gripper" />
+    <child
+      link="link_gripper_finger_left" />
+    <axis
+      xyz="0 0 1" />
+    <limit effort="100" lower="-0.6" upper="0.6" velocity="1.0"/>
+  </joint>
+  <link
+    name="link_gripper_fingertip_left">
+    <inertial>
+      <origin
+        xyz="0 0 0.008126"
+        rpy="0 0 0" />
+      <mass
+        value="0.003822" />
       <inertia
         ixx="0"
@@ -124,13 +178,66 @@
         iyy="0"
         iyz="0"
-        izz="0" />
-    </inertial>
-    <visual>
-      <origin
-        xyz="0 0 0"
-        rpy="0 0 0" />
-      <geometry>
-        <mesh
-          filename="package://stretch_description/meshes/link_gripper_finger_left.STL" scale="${scale_finger_length} 1.0 1.0"/>
+        izz="1E-06" />
+    </inertial>
+    <visual>
+      <origin
+        xyz="0 0 0"
+        rpy="0 0 0" />
+      <geometry>
+        <mesh
+          filename="package://stretch_description/meshes/link_gripper_fingertip_left.STL" />
+      </geometry>
+      <material
+        name="">
+        <color
+          rgba="0.250980392156863 0.250980392156863 0.250980392156863 1" />
+      </material>
+    </visual>
+    <collision>
+      <origin
+        xyz="0 0 0"
+        rpy="0 0 0" />
+      <geometry>
+        <mesh
+          filename="package://stretch_description/meshes/link_gripper_fingertip_left.STL" />
+      </geometry>
+    </collision>
+  </link>
+  <joint
+    name="joint_gripper_fingertip_left"
+    type="fixed">
+    <origin
+      xyz="${scale_finger_length * 0.19011} 0.014912 0"
+      rpy="-1.5708 -4.774E-15 -2.5545" />
+    <parent
+      link="link_gripper_finger_left" />
+    <child
+      link="link_gripper_fingertip_left" />
+    <axis
+      xyz="0 0 0" />
+  </joint>
+  <link
+    name="link_gripper_finger_right">
+    <inertial>
+      <origin
+        xyz="-0.093921 -0.011351 0"
+        rpy="0 0 0" />
+      <mass
+        value="0.06" />
+      <inertia
+        ixx="1.1E-05"
+        ixy="3.6E-05"
+        ixz="0"
+        iyy="0.000213"
+        iyz="0"
+        izz="0.000223" />
+    </inertial>
+    <visual>
+      <origin
+        xyz="0 0 0"
+        rpy="0 0 0" />
+      <geometry>
+        <mesh
+          filename="package://stretch_description/meshes/link_gripper_finger_right.STL" scale="${scale_finger_length} 1.0 1.0"/>
       </geometry>
       <material
@@ -146,18 +253,18 @@
       <geometry>
         <mesh
-          filename="package://stretch_description/meshes/link_gripper_finger_left.STL" scale="${scale_finger_length} 1.0 1.0"/>
-      </geometry>
-    </collision>
-  </link>
-  <joint
-    name="joint_gripper_finger_left"
+          filename="package://stretch_description/meshes/link_gripper_finger_right.STL" scale="${scale_finger_length} 1.0 1.0"/>
+      </geometry>
+    </collision>
+  </link>
+  <joint
+    name="joint_gripper_finger_right"
     type="revolute">
     <origin
-      xyz="-0.047231 -0.010151 -0.04679"
-      rpy="2.1762E-15 0.5236 3.1416" />
-    <parent
-      link="link_gripper" />
-    <child
-      link="link_gripper_finger_left" />
+      xyz="-0.047231 0.010049 -0.04679"
+      rpy="3.1416 -0.5236 1.2943E-15" />
+    <parent
+      link="link_gripper" />
+    <child
+      link="link_gripper_finger_right" />
     <axis
       xyz="0 0 1" />
@@ -165,11 +272,11 @@
   </joint>
   <link
-    name="link_gripper_fingertip_left">
-    <inertial>
-      <origin
-        xyz="-3.16381381648689E-08 -2.91408530639359E-09 0.00812579670381812"
-        rpy="0 0 0" />
-      <mass
-        value="0.00382159917455729" />
+    name="link_gripper_fingertip_right">
+    <inertial>
+      <origin
+        xyz="0 0 0.008126"
+        rpy="0 0 0" />
+      <mass
+        value="0.003822" />
       <inertia
         ixx="0"
@@ -178,112 +285,5 @@
         iyy="0"
         iyz="0"
-        izz="0" />
-    </inertial>
-    <visual>
-      <origin
-        xyz="0 0 0"
-        rpy="0 0 0" />
-      <geometry>
-        <mesh
-          filename="package://stretch_description/meshes/link_gripper_fingertip_left.STL" />
-      </geometry>
-      <material
-        name="">
-        <color
-          rgba="0.250980392156863 0.250980392156863 0.250980392156863 1" />
-      </material>
-    </visual>
-    <collision>
-      <origin
-        xyz="0 0 0"
-        rpy="0 0 0" />
-      <geometry>
-        <mesh
-          filename="package://stretch_description/meshes/link_gripper_fingertip_left.STL" />
-      </geometry>
-    </collision>
-  </link>
-  <joint
-    name="joint_gripper_fingertip_left"
-    type="fixed">
-    <origin
-      xyz="${scale_finger_length * 0.19011} 0.014912 0"
-      rpy="-1.5708 -4.774E-15 -2.5545" />
-    <parent
-      link="link_gripper_finger_left" />
-    <child
-      link="link_gripper_fingertip_left" />
-    <axis
-      xyz="0 0 0" />
-  </joint>
-  <link
-    name="link_gripper_finger_right">
-    <inertial>
-      <origin
-        xyz="-0.0945047483510099 -0.0124301080924345 0"
-        rpy="0 0 0" />
-      <mass
-        value="0.0476207785199481" />
-      <inertia
-        ixx="0"
-        ixy="0"
-        ixz="0"
-        iyy="0"
-        iyz="0"
-        izz="0" />
-    </inertial>
-    <visual>
-      <origin
-        xyz="0 0 0"
-        rpy="0 0 0" />
-      <geometry>
-        <mesh
-          filename="package://stretch_description/meshes/link_gripper_finger_right.STL" scale="${scale_finger_length} 1.0 1.0"/>
-      </geometry>
-      <material
-        name="">
-        <color
-          rgba="0.792156862745098 0.819607843137255 0.933333333333333 1" />
-      </material>
-    </visual>
-    <collision>
-      <origin
-        xyz="0 0 0"
-        rpy="0 0 0" />
-      <geometry>
-        <mesh
-          filename="package://stretch_description/meshes/link_gripper_finger_right.STL" scale="${scale_finger_length} 1.0 1.0"/>
-      </geometry>
-    </collision>
-  </link>
-  <joint
-    name="joint_gripper_finger_right"
-    type="revolute">
-    <origin
-      xyz="-0.047231 0.010049 -0.04679"
-      rpy="3.1416 -0.5236 1.2943E-15" />
-    <parent
-      link="link_gripper" />
-    <child
-      link="link_gripper_finger_right" />
-    <axis
-      xyz="0 0 1" />
-    <limit effort="100" lower="-0.6" upper="0.6" velocity="1.0"/>
-  </joint>
-  <link
-    name="link_gripper_fingertip_right">
-    <inertial>
-      <origin
-        xyz="2.59386303963494E-08 6.70949018566347E-09 0.00812579516130402"
-        rpy="0 0 0" />
-      <mass
-        value="0.00382160037319545" />
-      <inertia
-        ixx="0"
-        ixy="0"
-        ixz="0"
-        iyy="0"
-        iyz="0"
-        izz="0" />
+        izz="1E-06" />
     </inertial>
     <visual>

File: stretch_description/batch/mitski/urdf/stretch_laser_range_finder.xacro (robot description, xacro)
@@ -5,15 +5,15 @@
     <inertial>
       <origin
-        xyz="0 0 -0.000755956127492408"
+        xyz="0.011979 -0.000523 -0.01998"
         rpy="0 0 0" />
       <mass
-        value="0.0749979022894495" />
+        value="0.216007" />
       <inertia
-        ixx="0"
-        ixy="0"
-        ixz="0"
-        iyy="0"
-        iyz="0"
-        izz="0" />
+        ixx="9.5E-05"
+        ixy="2E-06"
+        ixz="-1.9E-05"
+        iyy="0.000184"
+        iyz="-1E-06"
+        izz="0.000216" />
     </inertial>
     <visual>

File: stretch_description/batch/mitski/urdf/stretch_main.xacro (robot description, xacro)
@@ -10,15 +10,15 @@
     <inertial>
       <origin
-        xyz="-0.11587 0.0019426 0.093621"
-        rpy="0 0 0" />
-      <mass
-        value="1.1912" />
-      <inertia
-        ixx="0.0034667"
-        ixy="-5.0568E-06"
-        ixz="0.00042861"
-        iyy="0.0052744"
-        iyz="-5.766E-05"
-        izz="0.0047945" />
+        xyz="-0.087526 -0.001626 0.081009"
+        rpy="0 0 0" />
+      <mass
+        value="17.384389" />
+      <inertia
+        ixx="0.160002"
+        ixy="0.006758"
+        ixz="0.004621"
+        iyy="0.138068"
+        iyz="0.002208"
+        izz="0.228992" />
     </inertial>
     <visual>
@@ -50,15 +50,15 @@
     <inertial>
       <origin
-        xyz="1.1719E-11 2.0783E-11 0.037544"
-        rpy="0 0 0" />
-      <mass
-        value="0.0042721" />
-      <inertia
-        ixx="0.001"
+        xyz="0 0 0.02765"
+        rpy="0 0 0" />
+      <mass
+        value="0.20773" />
+      <inertia
+        ixx="5.4E-05"
         ixy="0"
         ixz="0"
-        iyy="0.001"
+        iyy="5.4E-05"
         iyz="0"
-        izz="0.001" />
+        izz="5.1E-05" />
     </inertial>
     <visual>
@@ -104,15 +104,15 @@
     <inertial>
       <origin
-        xyz="-2.0783E-11 -1.1719E-11 -0.037544"
-        rpy="0 0 0" />
-      <mass
-        value="0.0042721" />
-      <inertia
-        ixx="0.001"
+        xyz="0 0 -0.02765"
+        rpy="0 0 0" />
+      <mass
+        value="0.20773" />
+      <inertia
+        ixx="5.4E-05"
         ixy="0"
         ixz="0"
-        iyy="0.001"
+        iyy="5.4E-05"
         iyz="0"
-        izz="0.001" />
+        izz="5.1E-05" />
     </inertial>
     <visual>
@@ -207,15 +207,15 @@
     <inertial>
       <origin
-        xyz="2.0817E-17 0.7075 -2.7756E-17"
-        rpy="0 0 0" />
-      <mass
-        value="1.8285" />
-      <inertia
-        ixx="0.0709854511954588"
-        ixy="-0.00433428742758457"
-        ixz="-0.000186110788697573"
-        iyy="0.000437922053342648"
-        iyz="-0.00288788257713431"
-        izz="0.071104808501661" />
+        xyz="0.000337 0.722201 0.002652"
+        rpy="0 0 0" />
+      <mass
+        value="1.764017" />
+      <inertia
+        ixx="0.291286"
+        ixy="0.004149"
+        ixz="-0.000174"
+        iyy="0.001226"
+        iyz="0.000354"
+        izz="0.291429" />
     </inertial>
     <visual>
@@ -260,15 +260,15 @@
     <inertial>
       <origin
-        xyz="-0.031727 0.038403 0.013361"
-        rpy="0 0 0" />
-      <mass
-        value="0.27218" />
-      <inertia
-        ixx="0.00052571"
-        ixy="0.00014899"
-        ixz="-1.9258E-05"
-        iyy="0.00030679"
-        iyz="-6.2451E-06"
-        izz="0.00037324" />
+        xyz="-0.020369 0.03438 0.02236"
+        rpy="0 0 0" />
+      <mass
+        value="1.987167" />
+      <inertia
+        ixx="0.006518"
+        ixy="-0.001539"
+        ixz="0.000371"
+        iyy="0.004464"
+        iyz="0.000392"
+        izz="0.008092" />
     </inertial>
     <visual>
@@ -317,15 +317,15 @@
     <inertial>
       <origin
-        xyz="-1.0146E-06 -1.9719E-05 -0.094738"
-        rpy="0 0 0" />
-      <mass
-        value="0.068095" />
-      <inertia
-        ixx="0.0001256"
-        ixy="-5.6914E-12"
-        ixz="6.0647E-09"
-        iyy="0.0001256"
-        iyz="1.1787E-07"
-        izz="1.1091E-10" />
+        xyz="-0.000168 -0.000254 -0.125235"
+        rpy="0 0 0" />
+      <mass
+        value="0.235626" />
+      <inertia
+        ixx="0.001518"
+        ixy="-1E-06"
+        ixz="3E-06"
+        iyy="0.001519"
+        iyz="3E-06"
+        izz="0.000176" />
     </inertial>
     <visual>
@@ -370,15 +370,15 @@
     <inertial>
       <origin
-        xyz="-5.13853606326845E-07 -1.99844969271112E-05 -0.0971104963726614"
-        rpy="0 0 0" />
-      <mass
-        value="0.0628927381893134" />
-      <inertia
-        ixx="0.001"
+        xyz="-1E-06 -0.000146 -0.11908"
+        rpy="0 0 0" />
+      <mass
+        value="0.146817" />
+      <inertia
+        ixx="0.001081"
         ixy="0"
         ixz="0"
-        iyy="0.001"
-        iyz="0"
-        izz="0.001" />
+        iyy="0.001081"
+        iyz="-1E-06"
+        izz="7.7E-05" />
     </inertial>
     <visual>
@@ -425,15 +425,15 @@
     <inertial>
       <origin
-        xyz="-5.17421949435687E-07 -2.02045301450349E-05 -0.0968815475684904"
-        rpy="0 0 0" />
-      <mass
-        value="0.0571386353275368" />
-      <inertia
-        ixx="0.001"
+        xyz="0 -7.1E-05 -0.115635"
+        rpy="0 0 0" />
+      <mass
+        value="0.130565" />
+      <inertia
+        ixx="0.000943"
         ixy="0"
         ixz="0"
-        iyy="0.001"
+        iyy="0.000943"
         iyz="0"
-        izz="0.001" />
+        izz="5.7E-05" />
     </inertial>
     <visual>
@@ -480,15 +480,15 @@
     <inertial>
       <origin
-        xyz="-5.257E-07 -2.0482E-05 -0.096543"
-        rpy="0 0 0" />
-      <mass
-        value="0.051382" />
-      <inertia
-        ixx="0.001"
+        xyz="-1E-06 -0.000121 -0.113457"
+        rpy="0 0 0" />
+      <mass
+        value="0.113658" />
+      <inertia
+        ixx="0.0008"
         ixy="0"
         ixz="0"
-        iyy="0.001"
+        iyy="0.0008"
         iyz="0"
-        izz="0.001" />
+        izz="4E-05" />
     </inertial>
     <visual>
@@ -535,15 +535,15 @@
     <inertial>
       <origin
-        xyz="0.0270582141286185 -0.00189876414654466 -0.0377809018481181"
-        rpy="0 0 0" />
-      <mass
-        value="0.085003260946398" />
-      <inertia
-        ixx="0.001"
-        ixy="0"
-        ixz="0"
-        iyy="0.001"
-        iyz="0"
-        izz="0.001" />
+        xyz="0.033681 -0.000847 -0.031723"
+        rpy="0 0 0" />
+      <mass
+        value="0.427734" />
+      <inertia
+        ixx="0.001689"
+        ixy="-2.8E-05"
+        ixz="0.000483"
+        iyy="0.002107"
+        iyz="-1.1E-05"
+        izz="0.000571" />
     </inertial>
     <visual>
@@ -590,15 +590,15 @@
     <inertial>
       <origin
-        xyz="2.20122392535771E-11 2.9317167880849E-05 -0.018966592644729"
-        rpy="0 0 0" />
-      <mass
-        value="0.0404746907425003" />
-      <inertia
-        ixx="0.001"
+        xyz="0 -3.9E-05 -0.016495"
+        rpy="0 0 0" />
+      <mass
+        value="0.054422" />
+      <inertia
+        ixx="9E-06"
         ixy="0"
         ixz="0"
-        iyy="0.001"
+        iyy="9E-06"
         iyz="0"
-        izz="0.001" />
+        izz="7E-06" />
     </inertial>
     <visual>
@@ -650,15 +650,15 @@
     <inertial>
       <origin
-        xyz="0.0406850995527703 0.0396956343318414 0.0226500246461012"
-        rpy="0 0 0" />
-      <mass
-        value="0.133027236718691" />
-      <inertia
-        ixx="0.001"
-        ixy="0"
-        ixz="0"
-        iyy="0.001"
-        iyz="0"
-        izz="0.001" />
+        xyz="0.047462 0.04451 0.016376"
+        rpy="0 0 0" />
+      <mass
+        value="0.681871" />
+      <inertia
+        ixx="0.001023"
+        ixy="0.000641"
+        ixz="6.6E-05"
+        iyy="0.002097"
+        iyz="6.5E-05"
+        izz="0.00281" />
     </inertial>
     <visual>
@@ -703,15 +703,15 @@
     <inertial>
       <origin
-        xyz="-0.000326562615178591 0.00850012613776489 0.000130487222982367"
-        rpy="0 0 0" />
-      <mass
-        value="0.0273764496535409" />
-      <inertia
-        ixx="0.001"
-        ixy="0"
-        ixz="0"
-        iyy="0.001"
-        iyz="0"
-        izz="0.001" />
+        xyz="-0.000422 0.013934 -0.0161"
+        rpy="0 0 0" />
+      <mass
+        value="0.062462" />
+      <inertia
+        ixx="4.1E-05"
+        ixy="-1E-06"
+        ixz="1E-06"
+        iyy="3.2E-05"
+        iyz="-1.5E-05"
+        izz="2.2E-05" />
     </inertial>
     <visual>
@@ -758,15 +758,15 @@
     <inertial>
       <origin
-        xyz="0.00704566394917504 -0.0212256210929691 0.0302058990060359"
-        rpy="0 0 0" />
-      <mass
-        value="0.090217113313934" />
-      <inertia
-        ixx="0.001"
-        ixy="0"
-        ixz="0"
-        iyy="0.001"
-        iyz="0"
-        izz="0.001" />
+        xyz="0.003907 -0.02418 0.030154"
+        rpy="0 0 0" />
+      <mass
+        value="0.283548" />
+      <inertia
+        ixx="0.000316"
+        ixy="-6E-06"
+        ixz="1E-06"
+        iyy="0.000143"
+        iyz="-2E-06"
+        izz="0.00031" />
     </inertial>
     <visual>

File: stretch_description/batch/mitski/urdf/stretch_respeaker.xacro (robot description, xacro)
@@ -5,15 +5,15 @@
     <inertial>
       <origin
-        xyz="-0.003809 -0.0023075 -0.012854"
+        xyz="-0.001594 -0.001282 -0.008098"
         rpy="0 0 0" />
       <mass
-        value="0.015643" />
+        value="0.025175" />
       <inertia
-        ixx="1.0075E-06"
-        ixy="-5.4396E-08"
-        ixz="-2.8652E-07"
-        iyy="1.0569E-06"
-        iyz="-1.8463E-07"
-        izz="1.1947E-07" />
+        ixx="1E-05"
+        ixy="2E-06"
+        ixz="1E-06"
+        iyy="1.2E-05"
+        iyz="0"
+        izz="1.5E-05" />
     </inertial>
     <visual>

File: stretch_description/urdf/cad_to_urdf/stretch_description_dex.xacro (robot description, xacro)
@@ -1,5 +1,6 @@
 <?xml version="1.0"?>
-<robot xmlns:xacro="http://www.ros.org/wiki/xacro" name="stretch">
-  <xacro:include filename="stretch_gripper.xacro" />
+<robot xmlns:xacro="http://www.ros.org/wiki/xacro" name="stretch_description">
+  <xacro:include filename="stretch_dex_wrist.xacro" />
+  <!--<xacro:include filename="stretch_gripper.xacro" /> -->
   <!--<xacro:include filename="stretch_gripper_with_puller.xacro" />-->
   <!--<xacro:include filename="stretch_dry_erase_marker.xacro" />-->
@@ -8,5 +9,4 @@
   <xacro:include filename="stretch_d435i.xacro" />
   <xacro:include filename="stretch_laser_range_finder.xacro" />
-  <xacro:include filename="stretch_base_imu.xacro" />
   <xacro:include filename="stretch_respeaker.xacro" />
 </robot>
